File: squelch_board.sch (KiCad schematic (older format))
At the start: 97 parts, among them P1 PWR, P2 DISC., P3 OUT, P4 CONN_02X04, P5 CONN-10033526-N3212LF, P6 CONN_01X05, P7 LPF, P8 NOISE, P9 DISC., Q1 MMBT2222A, U1 STM32F030F4P6, U2 Ricom R-786.5-0.5, U3 AP2202, U4 MCP6002, U5 MCP6002, U6 CP2105

Commit message: Upgrading schematic to current version of KiCad
Parts:
- C1, C10, C11, C12, C13, C14, C15, C16, C17, C18, C19, C2, C20, C21, C22, C23, C24, C25, C3, C4, C5, C6, C7, C8, C9: symbol C -> squelch_board-rescue:C
- D1, D2: symbol S1B -> squelch_board-rescue:S1B
- D10: symbol SP0503BAHT -> squelch_board-rescue:SP0503BAHT
- D11, D12, D13, D4, D5, D6, D7, D8, D9: symbol LED -> squelch_board-rescue:LED
- D3: symbol MMBD4148SE -> squelch_board-rescue:MMBD4148SE
- F1: symbol Fuse -> squelch_board-rescue:Fuse
- FB1, FB2: symbol FILTER -> squelch_board-rescue:FILTER
- MP1, MP2, MP3, MP4: symbol SCREW -> squelch_board-rescue:SCREW
- P1, P3: symbol CONN_01X03 -> squelch_board-rescue:CONN_01X03
- P2: symbol CONN_01X02 -> squelch_board-rescue:CONN_01X02
- P4: symbol CONN_02X04 -> squelch_board-rescue:CONN_02X04
- P5: symbol CONN-10033526-N3212LF -> squelch_board-rescue:CONN-10033526-N3212LF
- P6: symbol CONN_01X05 -> squelch_board-rescue:CONN_01X05
- P7, P8, P9: symbol CONN_COAXIAL -> squelch_board-rescue:CONN_COAXIAL
- Q1: symbol MMBT2222A -> squelch_board-rescue:MMBT2222A
- R1, R10, R11, R12, R13, R14, R15, R16, R17, R18, R19, R2, R20, R21, R22, R23, R24, R25, R26, R27, R28, R29, R3, R30, R31, R32, R33, R34, R4, R5, R6, R7, R8, R9: symbol R -> squelch_board-rescue:R
- TP1, TP2: symbol TEST -> squelch_board-rescue:TEST
- U1: symbol STM32F030F4P6 -> squelch_board-rescue:STM32F030F4P6
- U2: symbol LM7805CT -> squelch_board-rescue:LM7805CT
- U3: symbol APE8865U5-33-HF-3 -> squelch_board-rescue:APE8865U5-33-HF-3
- U4, U5: symbol MCP6002 -> squelch_board-rescue:MCP6002
- U6: symbol CP2105 -> squelch_board-rescue:CP2105

Commit message: Starting with rev 2.0 mods: Removing detector circuitry
Parts:
- removed C12: 0.01u, Capacitors_SMD:C_0603, symbol squelch_board-rescue:C
- removed C15: 0.0047u, Capacitors_SMD:C_0603, symbol squelch_board-rescue:C
- removed C16, C20: 470p, Capacitors_SMD:C_0603, symbol squelch_board-rescue:C
- removed D3: MMBD4148SE, smd-semi:SOT-23, symbol squelch_board-rescue:MMBD4148SE
- removed Q1: MMBT2222A, smd-semi:SOT-23, symbol squelch_board-rescue:MMBT2222A
- removed R11: 100, Resistors_SMD:R_0603, symbol squelch_board-rescue:R
- removed R14, R16, R18: 470k, Resistors_SMD:R_0603, symbol squelch_board-rescue:R
- removed R15: 680, Resistors_SMD:R_0603, symbol squelch_board-rescue:R
- removed R22: 0R, Resistors_SMD:R_0603, symbol squelch_board-rescue:R
- P8: value NOISE -> HPF
Connections:
- net HPF_OUT is gone; now on net NOISE: R13.1, R19.2, TP2.1, U5.1, U5.2 (-)
- net 3V3: now also U4.8 (V+)
- net GND: now also U4.4 (V-), U5.4 (V-), U5.5 (+)
- net NOISE: no longer U5.6 (-), U5.7
- net at C14.1, R17.2, R23.2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: now also U5.8 (V+)
- new net: U5.6 (-), U5.7
- no-connect marks 18 -> 14
Other:
- note added: "Can be used for\npower supply\nripple rejection."
- note removed: "Peak detector"
- note removed: "Populate either.\nCan be used for\npower supply\nripple rejection."
- moved on the sheet: C1, C10, C11, C13, C14, C17, C18, C19, C2, C21, C22, C23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

Commit message: Removing R23 (selector for OPA rail voltage and potential ripple rejection)
Parts:
- removed R23: 0R, Resistors_SMD:R_0603, symbol squelch_board-rescue:R
Connections:
- net 3V3: now also C14.1, R17.2, U5.8 (V+), U5.8 (V+)
Other:
- note removed: "Can be used for\npower supply\nripple rejection."
Changed lines of the file:
@@
 	1    0    0    -1
 $EndComp
-Text Label 7600 4450 0    60   ~ 0
+Text Label 7200 5125 0    60   ~ 0
 3V3
 $Comp
@@
 $EndComp
 $Comp
-L squelch_board-rescue:R R23
-U 1 1 589C7254
-P 7600 4600
-F 0 "R23" H 7670 4646 50  0000 L CNN
-F 1 "0R" H 7670 4555 50  0000 L CNN
-F 2 "Resistors_SMD:R_0603" V -2795 -125 50  0001 C CNN
-F 3 "" H -2725 -125 50  0001 C CNN
-F 4 "RES SMD 0 [0603]" H 7600 4600 60  0001 C CNN "BOM"
-	1    7600 4600
-	1    0    0    -1
-$EndComp
-$Comp
 L squelch_board-rescue:TEST TP1
 U 1 1 589CDADC
@@
 Wire Wire Line
 	5375 6075 5375 6125
-Wire Notes Line
-	7100 4775 7100 6450
 Wire Wire Line
 	4175 5575 4250 5575
@@
 	975  1800 900  1800
 Connection ~ 6550 5125
-Wire Notes Line
-	7175 4000 8025 4000
-Wire Notes Line
-	8025 4000 8025 4800
-Wire Notes Line
-	8025 4800 7175 4800
-Wire Notes Line
-	7175 4800 7175 4000
 Wire Wire Line
 	8175 3350 8625 3350
@@
 	7025 5675 7475 5675
 Wire Wire Line
-	7600 5125 7600 4750
-Wire Wire Line
-	6550 5125 7600 5125
-Wire Wire Line
 	7925 5550 7885 5550
 $Comp
@@
 	6300 5375 6300 5125
 Wire Wire Line
-	8125 5125 7600 5125
-Connection ~ 7600 5125
-Wire Wire Line
 	8125 5350 8125 5125
 $Comp
@@
 Text Label 6050 4000 0    60   ~ 0
 3V3
-Text Notes 7225 4300 0    60   ~ 0
-Can be used for\npower supply\nripple rejection.
+Wire Wire Line
+	6550 5125 8125 5125
 $EndSCHEMATC

Commit message: Renaming "HPF" to "NOISE" in schematic and on silk screen.
Parts:
- TP2: value HPF -> NOISE
Changed lines of the file:
@@
 P 2975 5875
 F 0 "TP2" H 3053 6015 50  0000 L CNN
-F 1 "HPF" H 3053 5924 50  0000 L CNN
+F 1 "NOISE" H 3053 5924 50  0000 L CNN
 F 2 "manuf:TESTPOINT-KEYSTONE-5018" H 375 -850 50  0001 C CNN
 F 3 "" H 375 -850 50  0001 C CNN

Commit message: Swapping out STM32F030F4P6 for STM32F070F6P
Parts:
- removed U1: STM32F030F4P6, IPC7351-Nominal:SOP65P640X120-20, symbol squelch_board-rescue:STM32F030F4P6
- added U1: STM32F070F6P, Package_SO:TSSOP-20_4.4x6.5mm_P0.65mm, symbol MCU_ST_STM32F0:STM32F070F6Px
Connections:
- net 3V3: now also U1.16 (VDD), U1.5 (VDDA)
- net AF_BUF: now also U1.7 (PA1)
- net AF_MUTE: now also U1.8 (PA2)
- net BOOT0: now also U1.1 (BOOT0)
- net GND: now also U1.15 (VSS)
- net LPF_OUT: now also U1.11 (PA5)
- net NOISE: now also U1.6 (PA0)
- net USB2uC: now also U1.18 (PA10/PA12)
- net uC10: now also U1.10 (PA4)
- net uC2: now also U1.2 (PF0)
- net uC2USB: now also U1.17 (PA9/PA11)
- net uC3: now also U1.3 (PF1)
- net uC9: now also U1.9 (PA3)
- net ~RST: now also U1.4 (NRST)
Other:
- note added: "STM32F030F4P6\nmay also work"
- moved on the sheet: C1, C2, R1
Changed lines of the file:
@@
 	1    0    0    -1
 $EndComp
-Text Notes 6100 2425 0    60   ~ 0
+Text Notes 6125 2425 0    60   ~ 0
 Todo:\n- Taper off\n- output divider\n- R2\n- 576-3193-1-ND LDO with smaller footprint
 Text Notes 550  1050 0    300  ~ 60
@@
 AF_BUF
 $Comp
-L squelch_board-rescue:STM32F030F4P6 U1
-U 1 1 58514CCA
-P 9550 1550
-F 0 "U1" H 9050 2400 50  0000 C CNN
-F 1 "STM32F030F4P6" H 9850 2400 50  0000 C CNN
-F 2 "IPC7351-Nominal:SOP65P640X120-20" H 9550 300 50  0001 C CNN
-F 3 "" H 9550 2600 50  0000 C CNN
-F 4 "DIST DIGIKEY 497-14044-5-ND" H 9550 500 50  0001 C CNN "BOM"
-	1    9550 1550
-	1    0    0    -1
-$EndComp
-$Comp
 L squelch_board-rescue:C C2
 U 1 1 58515408
-P 8175 1100
-F 0 "C2" H 8275 1175 50  0000 L CNN
-F 1 "0.1u" H 8275 1100 50  0000 L CNN
-F 2 "Capacitors_SMD:C_0603" H 8290 1009 50  0001 L CNN
-F 3 "" H 8175 1100 50  0000 C CNN
-F 4 "CAP MLCC 0.1uF 10% ≥X5R [0603]" H 8175 1100 60  0001 C CNN "BOM"
-	1    8175 1100
+P 8200 1475
+F 0 "C2" H 8300 1550 50  0000 L CNN
+F 1 "0.1u" H 8300 1475 50  0000 L CNN
+F 2 "Capacitors_SMD:C_0603" H 8315 1384 50  0001 L CNN
+F 3 "" H 8200 1475 50  0000 C CNN
+F 4 "CAP MLCC 0.1uF 10% ≥X5R [0603]" H 8200 1475 60  0001 C CNN "BOM"
+	1    8200 1475
 	1    0    0    -1
 $EndComp
@@
 L squelch_board-rescue:C C1
 U 1 1 585158BC
-P 7725 1100
-F 0 "C1" H 7825 1175 50  0000 L CNN
-F 1 "0.1u" H 7825 1100 50  0000 L CNN
-F 2 "Capacitors_SMD:C_0603" H 7840 1009 50  0001 L CNN
-F 3 "" H 7725 1100 50  0000 C CNN
-F 4 "CAP MLCC 0.1uF 10% ≥X5R [0603]" H 7725 1100 60  0001 C CNN "BOM"
-	1    7725 1100
+P 7750 1475
+F 0 "C1" H 7850 1550 50  0000 L CNN
+F 1 "0.1u" H 7850 1475 50  0000 L CNN
+F 2 "Capacitors_SMD:C_0603" H 7865 1384 50  0001 L CNN
+F 3 "" H 7750 1475 50  0000 C CNN
+F 4 "CAP MLCC 0.1uF 10% ≥X5R [0603]" H 7750 1475 60  0001 C CNN "BOM"
+	1    7750 1475
 	1    0    0    -1
 $EndComp
@@
 L squelch_board-rescue:GND #PWR019
 U 1 1 58515D2D
-P 7950 1250
-F 0 "#PWR019" H 7950 1000 50  0001 C CNN
-F 1 "GND" H 7955 1077 50  0001 C CNN
-F 2 "" H 7950 1250 50  0000 C CNN
-F 3 "" H 7950 1250 50  0000 C CNN
-	1    7950 1250
+P 7975 1625
+F 0 "#PWR019" H 7975 1375 50  0001 C CNN
+F 1 "GND" H 7980 1452 50  0001 C CNN
+F 2 "" H 7975 1625 50  0000 C CNN
+F 3 "" H 7975 1625 50  0000 C CNN
+	1    7975 1625
 	1    0    0    -1
 $EndComp
@@
 L squelch_board-rescue:GND #PWR020
 U 1 1 58516217
-P 8850 2350
-F 0 "#PWR020" H 8850 2100 50  0001 C CNN
-F 1 "GND" H 8855 2177 50  0001 C CNN
-F 2 "" H 8850 2350 50  0000 C CNN
-F 3 "" H 8850 2350 50  0000 C CNN
-	1    8850 2350
+P 9550 2225
+F 0 "#PWR020" H 9550 1975 50  0001 C CNN
+F 1 "GND" H 9555 2052 50  0001 C CNN
+F 2 "" H 9550 2225 50  0000 C CNN
+F 3 "" H 9550 2225 50  0000 C CNN
+	1    9550 2225
 	1    0    0    -1
 $EndComp
@@
 L squelch_board-rescue:R R1
 U 1 1 58516660
-P 8375 1500
-F 0 "R1" H 8445 1546 50  0000 L CNN
-F 1 "22k" H 8445 1455 50  0000 L CNN
-F 2 "Resistors_SMD:R_0603" V 8305 1500 50  0001 C CNN
-F 3 "" H 8375 1500 50  0000 C CNN
-F 4 "RES SMD 22k 1% [0603]" H 8375 1500 60  0001 C CNN "BOM"
-	1    8375 1500
+P 8575 1475
+F 0 "R1" H 8645 1521 50  0000 L CNN
+F 1 "22k" H 8645 1430 50  0000 L CNN
+F 2 "Resistors_SMD:R_0603" V 8505 1475 50  0001 C CNN
+F 3 "" H 8575 1475 50  0000 C CNN
+F 4 "RES SMD 22k 1% [0603]" H 8575 1475 60  0001 C CNN "BOM"
+	1    8575 1475
 	1    0    0    -1
 $EndComp
@@
 L squelch_board-rescue:GND #PWR021
 U 1 1 58517133
-P 8375 1650
-F 0 "#PWR021" H 8375 1400 50  0001 C CNN
-F 1 "GND" H 8380 1477 50  0001 C CNN
-F 2 "" H 8375 1650 50  0000 C CNN
-F 3 "" H 8375 1650 50  0000 C CNN
-	1    8375 1650
-	1    0    0    -1
-$EndComp
-Text Label 7725 950  0    60   ~ 0
+P 8575 1625
+F 0 "#PWR021" H 8575 1375 50  0001 C CNN
+F 1 "GND" H 8580 1452 50  0001 C CNN
+F 2 "" H 8575 1625 50  0000 C CNN
+F 3 "" H 8575 1625 50  0000 C CNN
+	1    8575 1625
+	1    0    0    -1
+$EndComp
+Text Label 7750 1325 0    60   ~ 0
 3V3
-Text Label 10300 1750 0    60   ~ 0
+Text Label 10350 1725 0    60   ~ 0
 uC2USB
-Text Label 10300 1850 0    60   ~ 0
+Text Label 10350 1825 0    60   ~ 0
 USB2uC
-Text Label 10300 850  0    60   ~ 0
+Text Label 10350 925  0    60   ~ 0
 NOISE
-Text Label 10300 950  0    60   ~ 0
+Text Label 10350 1025 0    60   ~ 0
 AF_BUF
-Text Label 10300 1350 0    60   ~ 0
+Text Label 10350 1425 0    60   ~ 0
 LPF_OUT
 $Comp
@@
 Connection ~ 4250 5575
 Wire Wire Line
-	7725 950  8175 950
-Connection ~ 8175 950
-Wire Wire Line
-	7725 1250 7950 1250
-Connection ~ 7950 1250
-Wire Wire Line
-	8850 850  8725 850
-Wire Wire Line
-	8725 850  8725 950
-Connection ~ 8725 950
-Wire Wire Line
-	8375 1350 8375 1150
+	7750 1325 8200 1325
+Wire Wire Line
+	7750 1625 7975 1625
+Connection ~ 7975 1625
+Wire Wire Line
+	8575 1325 8575 1125
 Wire Wire Line
 	2475 1800 2800 1800
@@
 Text Label 10350 3800 0    60   ~ 0
 USB2uC
-Text Label 8850 1350 2    60   ~ 0
+Text Label 9050 925  2    60   ~ 0
 ~RST
-Text Label 8850 1150 2    60   ~ 0
+Text Label 9050 1125 2    60   ~ 0
 BOOT0
 Text Label 10350 4150 0    60   ~ 0
@@
 Text Label 2050 7025 0    60   ~ 0
 uC10
-Text Label 8850 1550 2    60   ~ 0
+Text Label 9050 1725 2    60   ~ 0
 uC2
-Text Label 8850 1750 2    60   ~ 0
+Text Label 9050 1825 2    60   ~ 0
 uC3
-Text Label 10300 1150 0    60   ~ 0
+Text Label 10350 1225 0    60   ~ 0
 uC9
-Text Label 10300 1250 0    60   ~ 0
+Text Label 10350 1325 0    60   ~ 0
 uC10
 Wire Wire Line
-	8375 1150 8850 1150
+	8575 1125 9050 1125
 $Comp
 L squelch_board-rescue:C C23
@@
 Text Label 6875 3625 1    60   ~ 0
 AF_MUTE
-Text Label 10300 1050 0    60   ~ 0
+Text Label 10350 1125 0    60   ~ 0
 AF_MUTE
 $Comp
@@
 	-1   0    0    -1
 $EndComp
-NoConn ~ 10300 1450
-NoConn ~ 10300 1550
-NoConn ~ 10300 2050
-NoConn ~ 10300 2150
-NoConn ~ 10300 2350
+NoConn ~ 10350 1525
+NoConn ~ 10350 1625
+NoConn ~ 10350 1925
+NoConn ~ 10350 2025
+NoConn ~ 9050 2025
 NoConn ~ 10350 3500
 NoConn ~ 10350 3600
@@
 	4250 5575 4500 5575
 Wire Wire Line
-	8175 950  8725 950
-Wire Wire Line
-	7950 1250 8175 1250
-Wire Wire Line
-	8725 950  8850 950
+	7975 1625 8200 1625
 Wire Wire Line
 	5950 5575 6100 5575
@@
 Wire Wire Line
 	6550 5125 8125 5125
+Wire Wire Line
+	9650 725  9650 650
+Wire Wire Line
+	8200 650  8200 1325
+Wire Wire Line
+	8200 650  9550 650
+Connection ~ 8200 1325
+Connection ~ 9550 650
+Wire Wire Line
+	9550 650  9650 650
+Wire Wire Line
+	9550 725  9550 650
+$Comp
+L MCU_ST_STM32F0:STM32F070F6Px U1
+U 1 1 5EEC5F6B
+P 9750 1425
+F 0 "U1" H 9200 2100 50  0000 C CNN
+F 1 "STM32F070F6P" H 10025 2125 50  0000 C CNN
+F 2 "Package_SO:TSSOP-20_4.4x6.5mm_P0.65mm" H 9150 725 50  0001 R CNN
+F 3 "http://www.st.com/st-web-ui/static/active/en/resource/technical/document/datasheet/DM00141386.pdf" H 9750 1425 50  0001 C CNN
+	1    9750 1425
+	1    0    0    -1
+$EndComp
+Text Notes 8175 2050 0    60   ~ 0
+STM32F030F4P6\nmay also work
 $EndSCHEMATC

Commit message: Slight rearrangement of schematic, renaming nodes for consistency.
Connections:
- net AF_BUF renamed AF
- net AF_MUTE renamed MUTE
- net LPF_OUT renamed LPF
Other:
- moved on the sheet: C23, P3, P7, R2
Changed lines of the file:
@@
 	0    1    1    0
 $EndComp
-Text Label 6550 4300 0    60   ~ 0
-LPF_OUT
 $Comp
 L squelch_board-rescue:C C7
@@
 	-1   0    0    1
 $EndComp
-$Comp
-L squelch_board-rescue:APE8865U5-33-HF-3 U3
-U 1 1 577FD992
-P 5075 1850
-F 0 "U3" H 5075 2167 50  0000 C CNN
-F 1 "AP2202" H 5075 2076 50  0000 C CNN
-F 2 "TO_SOT_Packages_SMD:SOT-23-5" H 5075 2076 50  0001 C CIN
-F 3 "" H 5075 1850 50  0000 C CNN
-F 4 "DIST DIGIKEY AP2202K-3.3TRG1" H 5075 1850 60  0001 C CNN "BOM"
-	1    5075 1850
-	1    0    0    -1
-$EndComp
 NoConn ~ 5525 1950
 $Comp
@@
 Text Notes 4100 6425 0    60   ~ 0
 3rd order Butterworth Sallen-Key HPF, cutoff 7.5 kHz
-$Comp
-L squelch_board-rescue:GND #PWR013
-U 1 1 577F848C
-P 7500 3725
-F 0 "#PWR013" H 7500 3475 50  0001 C CNN
-F 1 "GND" H 7505 3552 50  0001 C CNN
-F 2 "" H 7500 3725 50  0000 C CNN
-F 3 "" H 7500 3725 50  0000 C CNN
-	1    7500 3725
-	1    0    0    -1
-$EndComp
 Text Notes 6125 2425 0    60   ~ 0
 Todo:\n- Taper off\n- output divider\n- R2\n- 576-3193-1-ND LDO with smaller footprint
@@
 $EndComp
 Text Label 3525 4200 0    60   ~ 0
-AF_BUF
+AF
 $Comp
 L squelch_board-rescue:C C2
@@
 $EndComp
 $Comp
-L squelch_board-rescue:R R2
-U 1 1 5851673E
-P 6700 3625
-F 0 "R2" V 6500 3550 50  0000 L CNN
-F 1 "0" V 6600 3550 50  0000 L CNN
-F 2 "Resistors_SMD:R_0603" V 6630 3625 50  0001 C CNN
-F 3 "" H 6700 3625 50  0000 C CNN
-F 4 "RES SMD 0 [0603]" V 6700 3625 60  0001 C CNN "BOM"
-	1    6700 3625
-	0    1    1    0
-$EndComp
-$Comp
 L squelch_board-rescue:GND #PWR021
 U 1 1 58517133
@@
 NOISE
 Text Label 10350 1025 0    60   ~ 0
-AF_BUF
+AF
 Text Label 10350 1425 0    60   ~ 0
-LPF_OUT
+LPF
 $Comp
 L squelch_board-rescue:S1B D2
@@
 $EndComp
 Text Label 2325 5875 3    60   ~ 0
-AF_BUF
+AF
 Text Label 2975 5875 3    60   ~ 0
 NOISE
@@
 $EndComp
 $Comp
-L squelch_board-rescue:GND #PWR028
-U 1 1 589DCF95
-P 7475 3150
-F 0 "#PWR028" H 7525 3200 50  0001 C CNN
-F 1 "GND" H 7480 2977 50  0001 C CNN
-F 2 "" H -1200 -825 50  0001 C CNN
-F 3 "" H -1200 -825 50  0001 C CNN
-	1    7475 3150
-	1    0    0    -1
-$EndComp
-$Comp
 L squelch_board-rescue:GND #PWR029
 U 1 1 589E0205
@@
 	6550 4300 6450 4300
 Wire Wire Line
-	6550 3625 6550 3775
-Wire Wire Line
 	6550 3775 6075 3775
 Wire Wire Line
@@
 Connection ~ 7600 2850
 Wire Wire Line
-	7350 3150 7475 3150
-Wire Wire Line
 	8950 4450 8850 4450
 Wire Wire Line
@@
 	8850 4550 8950 4550
 Connection ~ 8850 4550
-Connection ~ 7475 3150
 Wire Wire Line
 	10350 2850 10850 2850
@@
 Wire Wire Line
 	10675 3300 10350 3300
-$Comp
-L squelch_board-rescue:CONN_01X03 P3
-U 1 1 589E7E28
-P 7700 3625
-F 0 "P3" H 7618 3300 50  0000 C CNN
-F 1 "OUT" H 7618 3391 50  0000 C CNN
-F 2 "w_conn_mpt:mpt_0,5%2f3-2,54" H 400 725 50  0001 C CNN
-F 3 "" H 400 725 50  0001 C CNN
-F 4 "DIST DIGIKEY ED10562-ND" H 7700 3625 60  0001 C CNN "BOM"
-	1    7700 3625
-	1    0    0    1
-$EndComp
-Text Label 7500 3525 2    60   ~ 0
-NOISE
 Connection ~ 8350 3750
 Wire Wire Line
@@
 Text Label 2050 6825 0    60   ~ 0
 PTT
-Connection ~ 6550 3775
 $Comp
 L squelch_board-rescue:CP2105 U6
@@
 Wire Wire Line
 	8575 1125 9050 1125
-$Comp
-L squelch_board-rescue:C C23
-U 1 1 58A0A787
-P 7025 3625
-F 0 "C23" V 7225 3575 50  0000 L CNN
-F 1 "1u" V 7150 3575 50  0000 L CNN
-F 2 "Capacitors_SMD:C_0603" H 7063 3475 50  0001 C CNN
-F 3 "" H 7025 3625 50  0000 C CNN
-F 4 "CAP MLCC 1uF 10% 25V ≥X5R [0603]" H 7025 3625 60  0001 C CNN "BOM"
-	1    7025 3625
-	0    1    -1   0
-$EndComp
-Wire Wire Line
-	7175 3625 7325 3625
-Wire Wire Line
-	6875 3625 6850 3625
-Text Label 6875 3625 1    60   ~ 0
-AF_MUTE
 Text Label 10350 1125 0    60   ~ 0
-AF_MUTE
+MUTE
 $Comp
 L squelch_board-rescue:C C24
@@
 	1    0    0    -1
 $EndComp
-Wire Wire Line
-	7100 3825 7325 3825
-Wire Wire Line
-	7325 3825 7325 3625
-Connection ~ 7325 3625
-$Comp
-L squelch_board-rescue:GND #PWR047
-U 1 1 58A0FED8
-P 6950 4025
-F 0 "#PWR047" H 7000 4075 50  0001 C CNN
-F 1 "GND" H 6955 3852 50  0001 C CNN
-F 2 "" H -50 50  50  0001 C CNN
-F 3 "" H -50 50  50  0001 C CNN
-	1    6950 4025
-	-1   0    0    -1
-$EndComp
 $Comp
 L squelch_board-rescue:CONN_COAXIAL P8
@@
 	950  2725 950  3350
 Connection ~ 950  3350
-$Comp
-L squelch_board-rescue:CONN_COAXIAL P7
-U 1 1 58A10A59
-P 6950 3825
-F 0 "P7" H 7125 3825 50  0000 L CNN
-F 1 "LPF" H 7100 3750 50  0000 L CNN
-F 2 "local:MOLEX-0734152063" H 75  -75 50  0001 C CNN
-F 3 "" H 75  -75 50  0001 C CNN
-F 4 "DIST DIGIKEY WM3914CT-ND" H 6950 3825 60  0001 C CNN "BOM"
-	1    6950 3825
-	-1   0    0    -1
-$EndComp
 NoConn ~ 10350 1525
 NoConn ~ 10350 1625
@@
 	8850 4550 8850 4600
 Wire Wire Line
-	7475 3150 7600 3150
-Wire Wire Line
 	8350 3750 8350 4200
 Wire Wire Line
@@
 Wire Wire Line
 	1800 3350 2025 3350
-Wire Wire Line
-	7325 3625 7500 3625
 Wire Wire Line
 	950  3350 1025 3350
@@
 Text Notes 8175 2050 0    60   ~ 0
 STM32F030F4P6\nmay also work
+$Comp
+L squelch_board-rescue:GND #PWR013
+U 1 1 577F848C
+P 7875 4400
+F 0 "#PWR013" H 7875 4150 50  0001 C CNN
+F 1 "GND" H 7880 4227 50  0001 C CNN
+F 2 "" H 7875 4400 50  0000 C CNN
+F 3 "" H 7875 4400 50  0000 C CNN
+	1    7875 4400
+	1    0    0    -1
+$EndComp
+$Comp
+L squelch_board-rescue:R R2
+U 1 1 5851673E
+P 6875 4300
+F 0 "R2" V 6675 4225 50  0000 L CNN
+F 1 "0" V 6775 4225 50  0000 L CNN
+F 2 "Resistors_SMD:R_0603" V 6805 4300 50  0001 C CNN
+F 3 "" H 6875 4300 50  0000 C CNN
+F 4 "RES SMD 0 [0603]" V 6875 4300 60  0001 C CNN "BOM"
+	1    6875 4300
+	0    1    1    0
+$EndComp
+$Comp
+L squelch_board-rescue:GND #PWR028
+U 1 1 589DCF95
+P 7475 3150
+F 0 "#PWR028" H 7525 3200 50  0001 C CNN
+F 1 "GND" H 7480 2977 50  0001 C CNN
+F 2 "" H -1200 -825 50  0001 C CNN
+F 3 "" H -1200 -825 50  0001 C CNN
+	1    7475 3150
+	1    0    0    -1
+$EndComp
+$Comp
+L squelch_board-rescue:CONN_01X03 P3
+U 1 1 589E7E28
+P 8075 4300
+F 0 "P3" H 7993 3975 50  0000 C CNN
+F 1 "OUT" H 7993 4066 50  0000 C CNN
+F 2 "w_conn_mpt:mpt_0,5%2f3-2,54" H 775 1400 50  0001 C CNN
+F 3 "" H 775 1400 50  0001 C CNN
+F 4 "DIST DIGIKEY ED10562-ND" H 8075 4300 60  0001 C CNN "BOM"
+	1    8075 4300
+	1    0    0    1
+$EndComp
+Text Label 7875 4200 2    60   ~ 0
+NOISE
+$Comp
+L squelch_board-rescue:C C23
+U 1 1 58A0A787
+P 7425 4300
+F 0 "C23" V 7625 4250 50  0000 L CNN
+F 1 "1u" V 7550 4250 50  0000 L CNN
+F 2 "Capacitors_SMD:C_0603" H 7463 4150 50  0001 C CNN
+F 3 "" H 7425 4300 50  0000 C CNN
+F 4 "CAP MLCC 1uF 10% 25V ≥X5R [0603]" H 7425 4300 60  0001 C CNN "BOM"
+	1    7425 4300
+	0    1    -1   0
+$EndComp
+Wire Wire Line
+	7575 4300 7725 4300
+Wire Wire Line
+	7275 4300 7025 4300
+Text Label 7275 4300 2    60   ~ 0
+MUTE
+Wire Wire Line
+	7575 4500 7725 4500
+Wire Wire Line
+	7725 4500 7725 4300
+Connection ~ 7725 4300
+$Comp
+L squelch_board-rescue:GND #PWR047
+U 1 1 58A0FED8
+P 7425 4700
+F 0 "#PWR047" H 7475 4750 50  0001 C CNN
+F 1 "GND" H 7430 4527 50  0001 C CNN
+F 2 "" H 425 725 50  0001 C CNN
+F 3 "" H 425 725 50  0001 C CNN
+	1    7425 4700
+	-1   0    0    -1
+$EndComp
+$Comp
+L squelch_board-rescue:CONN_COAXIAL P7
+U 1 1 58A10A59
+P 7425 4500
+F 0 "P7" H 7600 4500 50  0000 L CNN
+F 1 "LPF" H 7575 4425 50  0000 L CNN
+F 2 "local:MOLEX-0734152063" H 550 600 50  0001 C CNN
+F 3 "" H 550 600 50  0001 C CNN
+F 4 "DIST DIGIKEY WM3914CT-ND" H 7425 4500 60  0001 C CNN "BOM"
+	1    7425 4500
+	-1   0    0    -1
+$EndComp
+Wire Wire Line
+	7725 4300 7875 4300
+Wire Wire Line
+	7350 3150 7475 3150
+Connection ~ 7475 3150
+Wire Wire Line
+	7475 3150 7600 3150
+Text Label 6550 4300 0    60   ~ 0
+LPF
+Wire Wire Line
+	6725 4300 6550 4300
+$Comp
+L squelch_board-rescue:APE8865U5-33-HF-3 U3
+U 1 1 577FD992
+P 5075 1850
+F 0 "U3" H 5075 2167 50  0000 C CNN
+F 1 "AP2202" H 5075 2076 50  0000 C CNN
+F 2 "TO_SOT_Packages_SMD:SOT-23-5" H 5075 2076 50  0001 C CIN
+F 3 "" H 5075 1850 50  0000 C CNN
+F 4 "DIST DIGIKEY AP2202K-3.3TRG1" H 5075 1850 60  0001 C CNN "BOM"
+	1    5075 1850
+	1    0    0    -1
+$EndComp
 $EndSCHEMATC

Commit message: Bumping version number to 2.0
Other:
- note added: "HB9UF Squelch Board Rev 2.0"
- note removed: "HB9UF Squelch Board Rev 1.3"
Changed lines of the file:
@@
 Todo:\n- Taper off\n- output divider\n- R2\n- 576-3193-1-ND LDO with smaller footprint
 Text Notes 550  1050 0    300  ~ 60
-HB9UF Squelch Board Rev 1.3
+HB9UF Squelch Board Rev 2.0
 $Comp
 L squelch_board-rescue:C C17
