File: squelch_board.kicad_pcb (KiCad board)
At the start: 2 copper layers, 50 x 50 mm, 92 parts, among them P1 PWR, P2 DISC., P3 OUT, P4 CONN_02X04, P5 CONN-10033526-N3212LF, P6 CONN_01X05, P7 LPF, P8 HPF, P9 DISC., U1 STM32F070F6P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

Commit message: Changing silk screen block diagram: brin pictogram
Brain pictogrm is licensed under a CC-BY license, jessie_vp is
attributed for the original work. Source:
https://thenounproject.com/term/brain/35201/
Parts:
- added G***: LOGO, local:brain, B.Cu at (137.0, 71.8)
- moved G*** 0.25 mm to (127.0, 90.5)
Routing:
- net GND: track 45.9 -> 46.6 mm, vias 87 -> 88

Commit message: Renaming "Squelch Board" to "HB9UF Smart Squelch"
Other:
- board text added: "HB9UF Smart Squelch Rev 2.0 Design by Matt Weyland, HB9FRV"
- board text removed: "HB9UF Squelch Board Rev 2.0 Design by Matt Weyland, HB9FRV"
Changed lines of the file:
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@@
   (gr_line (start 143.75 92.75) (end 124.75 92.75) (layer B.SilkS) (width 0.2))
   (gr_line (start 143.75 99.5) (end 143.75 92.75) (layer B.SilkS) (width 0.2))
-  (gr_text "HB9UF Squelch Board Rev 2.0\nDesign by Matt Weyland, HB9FRV" (at 144 102) (layer B.SilkS)
+  (gr_text "HB9UF Smart Squelch Rev 2.0\nDesign by Matt Weyland, HB9FRV" (at 144 102) (layer B.SilkS)
     (effects (font (size 0.75 0.75) (thickness 0.15)) (justify left mirror))
   )

Commit message: Fixing direction of power supply arrows on silk screen
Other:
- board text removed: "9 - 32 VDC"
Changed lines of the file:
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@@
       (xy 0.42418 -1.016)) (layer B.SilkS) (width 0.00254))
   )
+  (gr_text 6V5 (at 119.75 68.75 90) (layer B.SilkS)
+    (effects (font (size 1.5 1.5) (thickness 0.3)) (justify right mirror))
+  )
+  (gr_line (start 126.5 64.25) (end 118.25 64.25) (layer B.SilkS) (width 0.2))
   (gr_line (start 137 83.75) (end 137 86.25) (layer B.SilkS) (width 0.2))
   (gr_circle (center 137 85.5) (end 136.8 85.5) (layer B.SilkS) (width 0.2))
@@
     (effects (font (size 0.75 0.75) (thickness 0.15)))
   )
-  (gr_text "9 - 32\nVDC" (at 115.75 65.75) (layer B.SilkS)
+  (gr_text Vin (at 127.75 68.25 90) (layer B.SilkS)
     (effects (font (size 1.5 1.5) (thickness 0.3)) (justify right mirror))
   )
@@
   (gr_line (start 143.25 73.55) (end 143.25 70.05) (layer B.SilkS) (width 0.2))
   (gr_line (start 143.25 70.05) (end 143.25 70.05) (layer B.SilkS) (width 0.2))
-  (gr_line (start 123.25 68.25) (end 123.25 67) (layer B.SilkS) (width 0.2))
-  (gr_line (start 125.5 64.75) (end 123.25 67) (layer B.SilkS) (width 0.2))
+  (gr_line (start 118.25 68.5) (end 118.25 64.25) (layer B.SilkS) (width 0.2))
   (gr_line (start 127.5 73) (end 129 73) (layer B.SilkS) (width 0.2))
   (gr_line (start 129 64.75) (end 129 73) (layer B.SilkS) (width 0.2))
-  (gr_line (start 126.5 63.75) (end 125.5 64.75) (layer B.SilkS) (width 0.2))
-  (gr_line (start 126.5 62.5) (end 126.5 63.75) (layer B.SilkS) (width 0.2))
+  (gr_line (start 126.5 62.5) (end 126.5 64.25) (layer B.SilkS) (width 0.2))
   (gr_line (start 129 63.75) (end 129 64.75) (layer B.SilkS) (width 0.2))
   (gr_line (start 129 62.25) (end 129 63.75) (layer B.SilkS) (width 0.2))
@@
     (polygon
       (pts
-        (xy 123.25 69.136648) (xy 122.75 67.636648) (xy 123.75 67.636648)
+        (xy 126.5 61.5) (xy 127 63) (xy 126 63)
       )
     )
@@
     (polygon
       (pts
-        (xy 129 61.75) (xy 129.5 63.25) (xy 128.5 63.25)
-      )
-    )
+        (xy 127 73) (xy 128.5 72.5) (xy 128.5 73.5)
+      )
+    )
